Commit message: urdf for bot added

File: sac_bot/urdf/gazebo_plugin.xacro (robot description, xacro)
@@ -24,7 +24,7 @@
             <leftJoint>base_to_front_left_wheel</leftJoint>
             <rightJoint>base_to_front_right_wheel</rightJoint>
-            <wheelSeparation>0.2</wheelSeparation>
-            <wheelDiameter>0.12</wheelDiameter>
-            <torque>0.1</torque>
+            <wheelSeparation>0.1</wheelSeparation>
+            <wheelDiameter>0.06</wheelDiameter>
+            <torque>0.05</torque>
             <commandTopic>cmd_vel</commandTopic>
             <odometryTopic>odom</odometryTopic>
@@ -36,5 +36,5 @@
         <material>Gazebo/Blue</material>
 	    <sensor name="head_hokuyo_sensor" type="ray">
-	    	<pose>0.05 0 0 0 0 0</pose>
+	    	<pose>0.025 0 0 0 0 0</pose>
 	      	<visualize>false</visualize>
 	     	<update_rate>40</update_rate>

File: sac_bot/urdf/macros.xacro (robot description, xacro)
@@ -7,5 +7,5 @@
                 <origin rpy="1.57079632679 0 0" xyz="0 0 0"/>
                 <geometry>
-                <cylinder length="0.025" radius="0.06"/>
+                <cylinder length="0.0125" radius="0.03"/>
                 </geometry>
                 <material name="Black"/>
@@ -14,11 +14,11 @@
                 <origin rpy="0 1.507 1.507" xyz = "0 0 0"/>
                 <geometry>
-                    <cylinder length="0.025" radius="0.06"/>
+                    <cylinder length="0.0125" radius="0.03"/>
                 </geometry>
             </collision>
             <inertial>
                  <origin rpy="0 1.507 1.507" xyz = "0 0 0"/>
-                <mass value="0.2"/>
-                <xacro:cy_inertia mass="0.2" r="0.06" l="0.025" />
+                <mass value="0.1"/>
+                <xacro:cy_inertia mass="0.1" r="0.03" l="0.0125" />
             </inertial>
         </link>

File: sac_bot/urdf/robot.xacro (robot description, xacro)
@@ -6,20 +6,20 @@
     <!-- ************************ Base Link ******************************** -->
    <link name = "base_link">
-    <pose>0 0 0.1 0 0 0</pose>
+    <pose>0 0 0.05 0 0 0</pose>
     <visual>
-        <origin xyz="0 0 0.025" rpy="0 0 0" />
+        <origin xyz="0 0 0.0125" rpy="0 0 0" />
         <geometry>
-            <box size = "0.3 0.2 0.1"/>
+            <box size = "0.15 0.1 0.05"/>
         </geometry>
     </visual>
     <collision>
       <geometry>
-            <box size = "0.3 0.2 0.1"/>
+            <box size = "0.15 0.1 0.05"/>
         </geometry>
     </collision>
     <inertial>
       <origin xyz="0 0 0" rpy="0 0 0" />
-      <mass value="1"/>
-      <xacro:box_inertia mass="1" x="0.3" y="0.2" z="0.1" />
+      <mass value="0.5"/>
+      <xacro:box_inertia mass="0.5" x="0.15" y="0.1" z="0.05" />
     </inertial>
   </link>
@@ -31,11 +31,11 @@
     <inertial>
       <origin xyz="0 0 0" rpy="0 0 0"/>
-      <mass value="1"/>
-      <xacro:cy_inertia mass="1" r="0.075" l="0.025" />
+      <mass value="0.5"/>
+      <xacro:cy_inertia mass="0.5" r="0.0375" l="0.0125" />
     </inertial>
     <visual>
       <origin xyz="0 0 0" rpy="0 0 0"/>
       <geometry>
-        <cylinder radius="0.075" length="0.025"/>
+        <cylinder radius="0.0375" length="0.0125"/>
       </geometry>
       <material name="white"/>
@@ -44,10 +44,10 @@
       <origin xyz="0 0 0" rpy="0 0 0"/>
       <geometry>
-        <cylinder radius="0.075" length="0.025"/>
+        <cylinder radius="0.0375" length="0.0125"/>
       </geometry>
     </collision>
   </link>
   <joint name="joint_sensor_laser" type="fixed">
-     <origin xyz="0.15 0 0.025" rpy="0 0 0"/>
+     <origin xyz="0.075 0 0.0125" rpy="0 0 0"/>
      <parent link="base_link"/>
      <child link="sensor_laser"/>
@@ -58,5 +58,5 @@
 	    	<origin xyz="0 0 0" rpy="0 0 0"/>
 	      	<geometry>
-	    		<box size="0.1 0.2 0.2"/>
+	    		<box size="0.05 0.1 0.1"/>
 	      	</geometry>
 	    </collision>
@@ -64,5 +64,5 @@
 	    	<origin xyz="0 0 0" rpy="0 0 0"/>
 	      	<geometry>
-	    		<box size="0.05 0.2 0.05"/>
+	    		<box size="0.025 0.1 0.025"/>
 	      	</geometry>
 	      	<material name="crusta"/>
@@ -70,6 +70,6 @@
 		<inertial>
 			<origin xyz="0 0 0" />
-			<mass value="1"/>
-      <xacro:box_inertia mass="1" x="0.05" y="0.2" z="0.2"/>
+			<mass value="0.5"/>
+      <xacro:box_inertia mass="0.5" x="0.025" y="0.1" z="0.1"/>
 		</inertial>
 	</link>
@@ -77,14 +77,14 @@
 	    <parent link="base_link"/>
 	    <child link="camera"/>
-	    <origin xyz="0.1 0 0.1" rpy="0 0 0"/>
+	    <origin xyz="0.05 0 0.05" rpy="0 0 0"/>
 	</joint>
   <!-- ************************ Wheelz and Jointz ******************************** -->
   <xacro:wheelz name = "back_right_wheel_link"/>
-  <xacro:jointz name = "base_to_right_wheel" child = "back_right_wheel_link" origin_xyz = "-0.1 -0.1 0.0"/>
+  <xacro:jointz name = "base_to_right_wheel" child = "back_right_wheel_link" origin_xyz = "-0.05 -0.05 0.0"/>
   <xacro:wheelz name = "back_left_wheel_link"/>
-  <xacro:jointz name = "back_to_left_wheel" child = "back_left_wheel_link" origin_xyz = "-0.1 0.1 0.0"/>
+  <xacro:jointz name = "back_to_left_wheel" child = "back_left_wheel_link" origin_xyz = "-0.05 0.05 0.0"/>
   <xacro:wheelz name = "front_right_wheel_link"/>
-  <xacro:jointz name = "base_to_front_right_wheel" child = "front_right_wheel_link" origin_xyz = "0.1 -0.1 0.0"/>
+  <xacro:jointz name = "base_to_front_right_wheel" child = "front_right_wheel_link" origin_xyz = "0.05 -0.05 0.0"/>
   <xacro:wheelz name = "front_left_wheel_link"/>
-  <xacro:jointz name = "base_to_front_left_wheel" child = "front_left_wheel_link" origin_xyz = "0.1 0.1 0.0"/>
+  <xacro:jointz name = "base_to_front_left_wheel" child = "front_left_wheel_link" origin_xyz = "0.05 0.05 0.0"/>
 </robot>

Commit message: urdf updated

File: sac_bot/urdf/gazebo_plugin.xacro (robot description, xacro)
@@ -24,7 +24,7 @@
             <leftJoint>base_to_front_left_wheel</leftJoint>
             <rightJoint>base_to_front_right_wheel</rightJoint>
-            <wheelSeparation>0.1</wheelSeparation>
-            <wheelDiameter>0.06</wheelDiameter>
-            <torque>0.05</torque>
+            <wheelSeparation>0.075</wheelSeparation>
+            <wheelDiameter>0.045</wheelDiameter>
+            <torque>0.0375</torque>
             <commandTopic>cmd_vel</commandTopic>
             <odometryTopic>odom</odometryTopic>
@@ -36,5 +36,5 @@
         <material>Gazebo/Blue</material>
 	    <sensor name="head_hokuyo_sensor" type="ray">
-	    	<pose>0.025 0 0 0 0 0</pose>
+	    	<pose>0.01875 0 0 0 0 0</pose>
 	      	<visualize>false</visualize>
 	     	<update_rate>40</update_rate>

File: sac_bot/urdf/macros.xacro (robot description, xacro)
@@ -7,5 +7,5 @@
                 <origin rpy="1.57079632679 0 0" xyz="0 0 0"/>
                 <geometry>
-                <cylinder length="0.0125" radius="0.03"/>
+                <cylinder length="0.009375" radius="0.0225"/>
                 </geometry>
                 <material name="Black"/>
@@ -14,11 +14,11 @@
                 <origin rpy="0 1.507 1.507" xyz = "0 0 0"/>
                 <geometry>
-                    <cylinder length="0.0125" radius="0.03"/>
+                    <cylinder length="0.009375" radius="0.0225"/>
                 </geometry>
             </collision>
             <inertial>
                  <origin rpy="0 1.507 1.507" xyz = "0 0 0"/>
-                <mass value="0.1"/>
-                <xacro:cy_inertia mass="0.1" r="0.03" l="0.0125" />
+                <mass value="0.075"/>
+                <xacro:cy_inertia mass="0.075" r="0.0225" l="0.009375" />
             </inertial>
         </link>
@@ -26,5 +26,5 @@
     <macro name="jointz" params="name child origin_xyz">
         <joint name="${name}" type="continuous">
-            <axis xyz="0 1 0"/>
+            <axis xyz="0 0.75 0"/>
             <parent link="base_link"/>
             <child link="${child}"/>

File: sac_bot/urdf/robot.xacro (robot description, xacro)
@@ -6,20 +6,20 @@
     <!-- ************************ Base Link ******************************** -->
    <link name = "base_link">
-    <pose>0 0 0.05 0 0 0</pose>
+    <pose>0 0 0.0375 0 0 0</pose>
     <visual>
-        <origin xyz="0 0 0.0125" rpy="0 0 0" />
+        <origin xyz="0 0 0.009375" rpy="0 0 0" />
         <geometry>
-            <box size = "0.15 0.1 0.05"/>
+            <box size = "0.1125 0.075 0.0375"/>
         </geometry>
     </visual>
     <collision>
       <geometry>
-            <box size = "0.15 0.1 0.05"/>
+            <box size = "0.1125 0.075 0.0375"/>
         </geometry>
     </collision>
     <inertial>
       <origin xyz="0 0 0" rpy="0 0 0" />
-      <mass value="0.5"/>
-      <xacro:box_inertia mass="0.5" x="0.15" y="0.1" z="0.05" />
+      <mass value="0.375"/>
+      <xacro:box_inertia mass="0.375" x="0.1125" y="0.1" z="0.0375" />
     </inertial>
   </link>
@@ -31,11 +31,11 @@
     <inertial>
       <origin xyz="0 0 0" rpy="0 0 0"/>
-      <mass value="0.5"/>
-      <xacro:cy_inertia mass="0.5" r="0.0375" l="0.0125" />
+      <mass value="0.375"/>
+      <xacro:cy_inertia mass="0.375" r="0.028125" l="0.009375" />
     </inertial>
     <visual>
       <origin xyz="0 0 0" rpy="0 0 0"/>
       <geometry>
-        <cylinder radius="0.0375" length="0.0125"/>
+        <cylinder radius="0.028125" length="0.009375"/>
       </geometry>
       <material name="white"/>
@@ -44,10 +44,10 @@
       <origin xyz="0 0 0" rpy="0 0 0"/>
       <geometry>
-        <cylinder radius="0.0375" length="0.0125"/>
+        <cylinder radius="0.028125" length="0.009375"/>
       </geometry>
     </collision>
   </link>
   <joint name="joint_sensor_laser" type="fixed">
-     <origin xyz="0.075 0 0.0125" rpy="0 0 0"/>
+     <origin xyz="0.05625 0 0.009375" rpy="0 0 0"/>
      <parent link="base_link"/>
      <child link="sensor_laser"/>
@@ -58,5 +58,5 @@
 	    	<origin xyz="0 0 0" rpy="0 0 0"/>
 	      	<geometry>
-	    		<box size="0.05 0.1 0.1"/>
+	    		<box size="0.0375 0.075 0.075"/>
 	      	</geometry>
 	    </collision>
@@ -64,5 +64,5 @@
 	    	<origin xyz="0 0 0" rpy="0 0 0"/>
 	      	<geometry>
-	    		<box size="0.025 0.1 0.025"/>
+	    		<box size="0.01875 0.075 0.01875"/>
 	      	</geometry>
 	      	<material name="crusta"/>
@@ -70,6 +70,6 @@
 		<inertial>
 			<origin xyz="0 0 0" />
-			<mass value="0.5"/>
-      <xacro:box_inertia mass="0.5" x="0.025" y="0.1" z="0.1"/>
+			<mass value="0.375"/>
+      <xacro:box_inertia mass="0.375" x="0.01875" y="0.075" z="0.075"/>
 		</inertial>
 	</link>
@@ -77,14 +77,14 @@
 	    <parent link="base_link"/>
 	    <child link="camera"/>
-	    <origin xyz="0.05 0 0.05" rpy="0 0 0"/>
+	    <origin xyz="0.0375 0 0.0375" rpy="0 0 0"/>
 	</joint>
   <!-- ************************ Wheelz and Jointz ******************************** -->
   <xacro:wheelz name = "back_right_wheel_link"/>
-  <xacro:jointz name = "base_to_right_wheel" child = "back_right_wheel_link" origin_xyz = "-0.05 -0.05 0.0"/>
+  <xacro:jointz name = "base_to_right_wheel" child = "back_right_wheel_link" origin_xyz = "-0.0375 -0.0375 0.0"/>
   <xacro:wheelz name = "back_left_wheel_link"/>
-  <xacro:jointz name = "back_to_left_wheel" child = "back_left_wheel_link" origin_xyz = "-0.05 0.05 0.0"/>
+  <xacro:jointz name = "back_to_left_wheel" child = "back_left_wheel_link" origin_xyz = "-0.0375 0.0375 0.0"/>
   <xacro:wheelz name = "front_right_wheel_link"/>
-  <xacro:jointz name = "base_to_front_right_wheel" child = "front_right_wheel_link" origin_xyz = "0.05 -0.05 0.0"/>
+  <xacro:jointz name = "base_to_front_right_wheel" child = "front_right_wheel_link" origin_xyz = "0.0375 -0.0375 0.0"/>
   <xacro:wheelz name = "front_left_wheel_link"/>
-  <xacro:jointz name = "base_to_front_left_wheel" child = "front_left_wheel_link" origin_xyz = "0.05 0.05 0.0"/>
+  <xacro:jointz name = "base_to_front_left_wheel" child = "front_left_wheel_link" origin_xyz = "0.0375 0.0375 0.0"/>
 </robot>
